Commit message: debug of the controller and modify the model of robot and the qp

File: OpenBase/ROS/open_base/xacro/main.urdf.xacro (robot description, xacro)
@@ -20,5 +20,5 @@
 	<visual>
 		<geometry>
-			<mesh filename="package://open_base/mesh/base.stl" scale="5.0 5.0 15.0"/>
+			<mesh filename="package://open_base/mesh/base.stl" scale="5.0 5.0 5.0"/>
 		</geometry>
 		<material name="base_material">
@@ -28,5 +28,5 @@
 	<collision>
 		<geometry>
-			<mesh filename="package://open_base/mesh/base.stl" scale="5.0 5.0 15.0"/>
+			<mesh filename="package://open_base/mesh/base.stl" scale="5.0 5.0 5.0"/>
 		</geometry>
 	</collision>
